File: kibod-01.kicad_pcb (KiCad board)
At the start: 2 copper layers, 312.8 x 87.8 mm, 87 parts, among them J1 02x05, J2 02x05, U1 ProMicro

Commit message: add gerber
Other:
- board size 312.8 x 87.8 mm -> 312.8 x 87.6 mm
Changed lines of the file:
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@@
   (gr_line (start 139.7 103.632) (end 136.271 123.317) (layer "Edge.Cuts") (width 0.05))
   (gr_line (start 297.572127 60.96) (end 287.412127 119.38) (layer "Edge.Cuts") (width 0.05))
-  (gr_line (start 230.262127 36.83) (end 230.262127 39.37) (layer "Edge.Cuts") (width 0.05))
-  (gr_line (start 184.542127 36.83) (end 207.402127 38.1) (layer "Edge.Cuts") (width 0.05))
-  (gr_line (start 184.542127 36.83) (end 184.542127 38.1) (layer "Edge.Cuts") (width 0.05))
-  (gr_line (start 230.262127 39.37) (end 253.122127 41.91) (layer "Edge.Cuts") (width 0.05))
+  (gr_line (start 229.362 37.084) (end 229.108 39.497) (layer "Edge.Cuts") (width 0.05))
+  (gr_line (start 185.166 37.211) (end 208.788 38.1) (layer "Edge.Cuts") (width 0.05))
+  (gr_line (start 185.166 37.211) (end 185.166 38.227) (layer "Edge.Cuts") (width 0.05))
+  (gr_line (start 229.108 39.497) (end 252.603 42.037) (layer "Edge.Cuts") (width 0.05))
   (gr_line (start 265.822127 115.57) (end 245.502127 113.03) (layer "Edge.Cuts") (width 0.05))
-  (gr_line (start 253.122127 41.91) (end 251.852127 53.34) (layer "Edge.Cuts") (width 0.05))
+  (gr_line (start 252.603 42.037) (end 251.46 53.34) (layer "Edge.Cuts") (width 0.05))
   (gr_line (start 184.542127 119.38) (end 165.492127 120.65) (layer "Edge.Cuts") (width 0.05))
   (gr_line (start 203.592127 118.11) (end 184.542127 119.38) (layer "Edge.Cuts") (width 0.05))
@@
   (gr_line (start 142.367 38.1) (end 162.952127 38.1) (layer "Edge.Cuts") (width 0.05))
   (gr_line (start 165.492127 120.65) (end 146.177 123.317) (layer "Edge.Cuts") (width 0.05))
-  (gr_line (start 207.402127 35.56) (end 230.262127 36.83) (layer "Edge.Cuts") (width 0.05))
+  (gr_line (start 208.915 35.814) (end 229.362 37.084) (layer "Edge.Cuts") (width 0.05))
   (gr_line (start 275.982127 57.15) (end 297.572127 60.96) (layer "Edge.Cuts") (width 0.05))
-  (gr_line (start 207.402127 38.1) (end 207.402127 35.56) (layer "Edge.Cuts") (width 0.05))
-  (gr_line (start 251.852127 53.34) (end 275.982127 57.15) (layer "Edge.Cuts") (width 0.05))
+  (gr_line (start 208.788 38.1) (end 208.915 35.814) (layer "Edge.Cuts") (width 0.05))
+  (gr_line (start 251.46 53.34) (end 275.982127 57.15) (layer "Edge.Cuts") (width 0.05))
   (gr_line (start 142.632127 103.632) (end 146.177 123.317) (layer "Edge.Cuts") (width 0.05))
-  (gr_line (start 162.952127 38.1) (end 184.542127 38.1) (layer "Edge.Cuts") (width 0.05))
+  (gr_line (start 162.952127 38.1) (end 185.166 38.227) (layer "Edge.Cuts") (width 0.05))
   (gr_line (start 142.367 102.489) (end 142.367 38.1) (layer "Edge.Cuts") (width 0.05))
   (gr_line (start 203.592127 118.11) (end 245.502127 113.03) (layer "Edge.Cuts") (width 0.05))
-  (gr_line (start 119.38 38.1) (end 97.79 38.1) (layer "Edge.Cuts") (width 0.05))
+  (gr_line (start 119.38 38.1) (end 96.774 38.227) (layer "Edge.Cuts") (width 0.05))
   (gr_line (start 139.954 102.489) (end 142.367 102.489) (layer "Edge.Cuts") (width 0.05))
   (gr_line (start -5.08 119.38) (end 16.51 115.57) (layer "Edge.Cuts") (width 0.05))
@@
   (gr_line (start 97.79 119.38) (end 116.84 120.65) (layer "Edge.Cuts") (width 0.05))
   (gr_line (start 139.954 102.489) (end 139.954 38.1) (layer "Edge.Cuts") (width 0.05))
-  (gr_line (start 52.07 39.37) (end 29.21 41.91) (layer "Edge.Cuts") (width 0.05))
-  (gr_line (start 74.93 38.1) (end 74.93 35.56) (layer "Edge.Cuts") (width 0.05))
+  (gr_line (start 52.705 39.37) (end 29.845 41.91) (layer "Edge.Cuts") (width 0.05))
+  (gr_line (start 73.533 37.846) (end 73.406 35.687) (layer "Edge.Cuts") (width 0.05))
   (gr_line (start -15.24 60.96) (end -5.08 119.38) (layer "Edge.Cuts") (width 0.05))
   (gr_line (start 16.51 115.57) (end 36.83 113.03) (layer "Edge.Cuts") (width 0.05))
-  (gr_line (start 29.21 41.91) (end 30.48 53.34) (layer "Edge.Cuts") (width 0.05))
-  (gr_line (start 52.07 36.83) (end 52.07 39.37) (layer "Edge.Cuts") (width 0.05))
+  (gr_line (start 29.972 42.164) (end 31.115 53.213) (layer "Edge.Cuts") (width 0.05))
+  (gr_line (start 52.578 37.084) (end 52.705 39.37) (layer "Edge.Cuts") (width 0.05))
   (gr_line (start 78.74 118.11) (end 36.83 113.03) (layer "Edge.Cuts") (width 0.05))
-  (gr_line (start 74.93 35.56) (end 52.07 36.83) (layer "Edge.Cuts") (width 0.05))
-  (gr_line (start 97.79 36.83) (end 97.79 38.1) (layer "Edge.Cuts") (width 0.05))
-  (gr_line (start 30.48 53.34) (end 6.35 57.15) (layer "Edge.Cuts") (width 0.05))
-  (gr_line (start 97.79 36.83) (end 74.93 38.1) (layer "Edge.Cuts") (width 0.05))
+  (gr_line (start 73.406 35.687) (end 52.578 37.084) (layer "Edge.Cuts") (width 0.05))
+  (gr_line (start 96.774 37.211) (end 96.774 38.227) (layer "Edge.Cuts") (width 0.05))
+  (gr_line (start 31.115 53.213) (end 6.35 57.15) (layer "Edge.Cuts") (width 0.05))
+  (gr_line (start 96.774 37.211) (end 73.533 37.846) (layer "Edge.Cuts") (width 0.05))
   (gr_line (start 116.84 120.65) (end 136.271 123.317) (layer "Edge.Cuts") (width 0.05))
   (gr_line (start 78.74 118.11) (end 97.79 119.38) (layer "Edge.Cuts") (width 0.05))

Commit message: add copper layer
Routing:
- added copper zone on B.Cu, net (none)
- added copper zone on F.Cu, net (none)
Other:
- outline, holes or cut-outs redrawn
Changed lines of the file:
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@@
   (gr_line (start -15.24 60.96) (end -5.08 119.38) (layer "Edge.Cuts") (width 0.05))
   (gr_line (start 16.51 115.57) (end 36.83 113.03) (layer "Edge.Cuts") (width 0.05))
-  (gr_line (start 29.972 42.164) (end 31.115 53.213) (layer "Edge.Cuts") (width 0.05))
+  (gr_line (start 29.845 41.91) (end 31.115 53.213) (layer "Edge.Cuts") (width 0.05))
   (gr_line (start 52.578 37.084) (end 52.705 39.37) (layer "Edge.Cuts") (width 0.05))
   (gr_line (start 78.74 118.11) (end 36.83 113.03) (layer "Edge.Cuts") (width 0.05))
@@
   (gr_line (start 78.74 118.11) (end 97.79 119.38) (layer "Edge.Cuts") (width 0.05))
   (gr_line (start 139.7 103.632) (end 142.632127 103.632) (layer "Edge.Cuts") (width 0.05))
+  (gr_text "github.com/GreenMashedPotato/kibod-01" (at 224.155 114.3 7) (layer "B.SilkS")
+    (effects (font (size 1 1) (thickness 0.15)) (justify mirror))
+  )
+  (gr_text "Kibod-01 by Michael G" (at 58.42 114.3 -6) (layer "B.SilkS")
+    (effects (font (size 1 1) (thickness 0.15)) (justify mirror))
+  )
   (gr_text "github.com/GreenMashedPotato/kibod-01" (at 224.155 114.3 7) (layer "F.SilkS")
     (effects (font (size 1 1) (thickness 0.15)))
@@
   (segment (start 111.74 44.74) (end 117.13 44.74) (width 0.25) (layer "F.Cu") (net 65))
   (segment (start 117.13 44.74) (end 118.11 45.72) (width 0.25) (layer "F.Cu") (net 65))
+  (zone (net 0) (net_name "") (layer "F.Cu") (hatch none 0.508)
+    (connect_pads (clearance 0.508))
+    (min_thickness 0.254) (filled_areas_thickness no)
+    (fill yes (thermal_gap 0.508) (thermal_bridge_width 0.508))
+    (polygon
+      (pts
+        (xy 73.533 37.846)
+        (xy 96.774 37.211)
+        (xy 96.774 38.227)
+        (xy 139.954 38.1)
+        (xy 139.954 102.489)
+        (xy 142.367 102.489)
+        (xy 142.367 38.1)
+        (xy 185.166 38.227)
+        (xy 185.166 37.211)
+        (xy 208.788 38.1)
+        (xy 208.915 35.814)
+        (xy 229.362 37.084)
+        (xy 229.108 39.497)
+        (xy 252.603 42.037)
+        (xy 251.46 53.34)
+        (xy 297.434 60.96)
+        (xy 297.561 60.96)
+        (xy 287.401 119.38)
+        (xy 265.938 115.57)
+        (xy 245.491 113.03)
+        (xy 203.454 118.11)
+        (xy 165.354 120.65)
+        (xy 146.177 123.317)
+        (xy 142.621 103.632)
+        (xy 139.7 103.632)
+        (xy 136.271 123.317)
+        (xy 116.84 120.65)
+        (xy 78.613 118.11)
+        (xy 36.957 113.03)
+        (xy 16.637 115.57)
+        (xy -5.207 119.38)
+        (xy -15.24 60.96)
+        (xy 31.115 53.213)
+        (xy 29.845 41.91)
+        (xy 52.705 39.37)
+        (xy 52.578 37.084)
+        (xy 73.406 35.687)
+      )
+    )
+  )
+  (zone (net 0) (net_name "") (layer "B.Cu") (hatch edge 0.508)
+    (connect_pads (clearance 0.508))
+    (min_thickness 0.254) (filled_areas_thickness no)
+    (fill yes (thermal_gap 0.508) (thermal_bridge_width 0.508))
+    (polygon
+      (pts
+        (xy 73.533 37.846)
+        (xy 96.774 37.211)
+        (xy 96.774 38.227)
+        (xy 139.954 38.1)
+        (xy 139.954 102.489)
+        (xy 142.367 102.489)
+        (xy 142.367 38.1)
+        (xy 185.166 38.227)
+        (xy 185.166 37.211)
+        (xy 208.788 38.1)
+        (xy 208.915 35.814)
+        (xy 229.362 37.084)
+        (xy 229.108 39.497)
+        (xy 252.603 42.037)
+        (xy 251.466756 53.299136)
+        (xy 297.567756 60.919136)
+        (xy 297.561 60.96)
+        (xy 287.401 119.38)
+        (xy 265.938 115.57)
+        (xy 245.618 113.03)
+        (xy 245.491 113.03)
+        (xy 203.454 118.11)
+        (xy 165.481 120.65)
+        (xy 146.304 123.317)
+        (xy 146.177 123.317)
+        (xy 142.621 103.632)
+        (xy 139.7 103.632)
+        (xy 136.271 123.19)
+        (xy 136.271 123.317)
+        (xy 116.84 120.65)
+        (xy 78.74 118.11)
+        (xy 36.83 113.03)
+        (xy 16.51 115.57)
+        (xy -4.953 119.38)
+        (xy -5.08 119.38)
+        (xy -15.24 60.96)
+        (xy 31.115 53.213)
+        (xy 29.845 41.91)
+        (xy 52.705 39.37)
+        (xy 52.578 37.084)
+        (xy 73.406 35.687)
+      )
+    )
+  )
 )

Commit message: fix minor issues
Other:
- outline, holes or cut-outs redrawn
Changed lines of the file:
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@@
   (gr_line (start 142.632127 103.632) (end 146.177 123.317) (layer "Edge.Cuts") (width 0.05))
   (gr_line (start 162.952127 38.1) (end 185.166 38.227) (layer "Edge.Cuts") (width 0.05))
-  (gr_line (start 142.367 102.489) (end 142.367 38.1) (layer "Edge.Cuts") (width 0.05))
+  (gr_line (start 142.367 102.235) (end 142.367 38.1) (layer "Edge.Cuts") (width 0.05))
   (gr_line (start 203.592127 118.11) (end 245.502127 113.03) (layer "Edge.Cuts") (width 0.05))
   (gr_line (start 119.38 38.1) (end 96.774 38.227) (layer "Edge.Cuts") (width 0.05))
-  (gr_line (start 139.954 102.489) (end 142.367 102.489) (layer "Edge.Cuts") (width 0.05))
+  (gr_line (start 139.954 102.235) (end 142.367 102.235) (layer "Edge.Cuts") (width 0.05))
   (gr_line (start -5.08 119.38) (end 16.51 115.57) (layer "Edge.Cuts") (width 0.05))
   (gr_line (start 6.35 57.15) (end -15.24 60.96) (layer "Edge.Cuts") (width 0.05))
   (gr_line (start 97.79 119.38) (end 116.84 120.65) (layer "Edge.Cuts") (width 0.05))
-  (gr_line (start 139.954 102.489) (end 139.954 38.1) (layer "Edge.Cuts") (width 0.05))
+  (gr_line (start 139.954 102.235) (end 139.954 38.1) (layer "Edge.Cuts") (width 0.05))
   (gr_line (start 52.705 39.37) (end 29.845 41.91) (layer "Edge.Cuts") (width 0.05))
   (gr_line (start 73.533 37.846) (end 73.406 35.687) (layer "Edge.Cuts") (width 0.05))
@@
   (segment (start 146.550055 109.218354) (end 145.220527 110.547882) (width 0.25) (layer "F.Cu") (net 44))
   (segment (start 50.657976 73.660001) (end 122.34 73.66) (width 0.25) (layer "F.Cu") (net 45))
-  (segment (start 144.976064 103.066064) (end 151.522127 96.52) (width 0.25) (layer "F.Cu") (net 45))
+  (segment (start 133.35 97.014988) (end 133.35 95.25) (width 0.25) (layer "F.Cu") (net 45))
   (segment (start 122.34 73.66) (end 138.43 57.57) (width 0.25) (layer "F.Cu") (net 45))
   (segment (start 250.936162 91.157625) (end 268.079752 91.157625) (width 0.25) (layer "F.Cu") (net 45))
   (segment (start 268.079752 91.157625) (end 274.12006 97.197933) (width 0.25) (layer "F.Cu") (net 45))
-  (segment (start 144.822118 103.22001) (end 144.976064 103.066064) (width 0.25) (layer "F.Cu") (net 45))
   (segment (start 1.726729 94.793271) (end 29.511268 94.793271) (width 0.25) (layer "F.Cu") (net 45))
   (segment (start 148.380221 96.52) (end 145.917289 94.057068) (width 0.25) (layer "F.Cu") (net 45))
+  (segment (start 145.293564 102.748564) (end 151.522127 96.52) (width 0.25) (layer "F.Cu") (net 45))
   (segment (start 29.517987 94.79999) (end 50.657976 73.660001) (width 0.25) (layer "F.Cu") (net 45))
+  (segment (start 143.058994 102.926994) (end 145.115134 102.926994) (width 0.25) (layer "F.Cu") (net 45))
   (segment (start 152.602907 77.01999) (end 236.798528 77.019991) (width 0.25) (layer "F.Cu") (net 45))
   (segment (start 279.285926 97.197933) (end 281.74006 99.652067) (width 0.25) (layer "F.Cu") (net 45))
@@
   (segment (start 281.74006 99.652067) (end 281.74006 102.980183) (width 0.25) (layer "F.Cu") (net 45))
   (segment (start 150.252127 96.52) (end 148.380221 96.52) (width 0.25) (layer "F.Cu") (net 45))
-  (segment (start 144.822117 103.22001) (end 144.976064 103.066064) (width 0.25) (layer "F.Cu") (net 45))
+  (segment (start 143.058994 102.926994) (end 139.262006 102.926994) (width 0.25) (layer "F.Cu") (net 45))
+  (segment (start 145.115134 102.926994) (end 145.293564 102.748564) (width 0.25) (layer "F.Cu") (net 45))
   (segment (start 145.91729 83.705607) (end 152.602907 77.01999) (width 0.25) (layer "F.Cu") (net 45))
-  (segment (start 139.555022 103.22001) (end 144.822118 103.22001) (width 0.25) (layer "F.Cu") (net 45))
-  (segment (start 133.35 95.25) (end 133.35 97.014988) (width 0.25) (layer "F.Cu") (net 45))
+  (segment (start 143.185994 102.926994) (end 143.058994 102.926994) (width 0.25) (layer "F.Cu") (net 45))
   (segment (start -0.003812 104.63077) (end -0.003812 96.523812) (width 0.25) (layer "F.Cu") (net 45))
   (segment (start 29.511268 94.793271) (end 29.517987 94.79999) (width 0.25) (layer "F.Cu") (net 45))
+  (segment (start 139.262006 102.926994) (end 133.35 97.014988) (width 0.25) (layer "F.Cu") (net 45))
   (segment (start 274.12006 97.197933) (end 279.285926 97.197933) (width 0.25) (layer "F.Cu") (net 45))
-  (segment (start 133.35 97.014988) (end 139.555022 103.22001) (width 0.25) (layer "F.Cu") (net 45))
   (segment (start 236.798528 77.019991) (end 250.936162 91.157625) (width 0.25) (layer "F.Cu") (net 45))
   (segment (start 151.522127 96.52) (end 151.522127 95.25) (width 0.25) (layer "F.Cu") (net 45))
@@
   (segment (start 111.74 44.74) (end 117.13 44.74) (width 0.25) (layer "F.Cu") (net 65))
   (segment (start 117.13 44.74) (end 118.11 45.72) (width 0.25) (layer "F.Cu") (net 65))
-  (zone (net 0) (net_name "") (layer "F.Cu") (hatch none 0.508)
+  (zone (net 0) (net_name "") (layer "F.Cu") (hatch edge 0.508)
     (connect_pads (clearance 0.508))
     (min_thickness 0.254) (filled_areas_thickness no)
@@
         (xy 96.774 38.227)
         (xy 139.954 38.1)
-        (xy 139.954 102.489)
-        (xy 142.367 102.489)
+        (xy 139.954 102.235)
+        (xy 142.367 102.235)
         (xy 142.367 38.1)
         (xy 185.166 38.227)
@@
     )
   )
-  (zone (net 0) (net_name "") (layer "B.Cu") (hatch edge 0.508)
+  (zone (net 0) (net_name "") (layers F&B.Cu) (hatch edge 0.508)
     (connect_pads (clearance 0.508))
     (min_thickness 0.254) (filled_areas_thickness no)
@@
         (xy 96.774 38.227)
         (xy 139.954 38.1)
-        (xy 139.954 102.489)
-        (xy 142.367 102.489)
+        (xy 139.954 102.235)
+        (xy 142.367 102.235)
         (xy 142.367 38.1)
         (xy 185.166 38.227)
