File: Mirrored/kibod-01.kicad_sch (KiCad schematic)
At the start: 46 parts, among them J1 02x05, J2 02x05, U1 ProMicro, U2 trrs

Commit message: fixed non reversible holes
Parts:
- K-0-0, K-0-1, K-0-2, K-0-3, K-0-4, K-0-5, K-1-0, K-1-1, K-1-2, K-1-3, K-1-4, K-1-5, K-2-0, K-2-1, K-2-2, K-2-3, K-2-4, K-2-5, K-3-3, K-3-4, K-3-5: footprint footprints:100-minimal-no-3d -> footprints:100-dual
