File: Mirrored Rev2/kibod-01-mirrored-rev2.kicad_sch (KiCad schematic)
At the start: 45 parts, among them J1 02x05, J2 02x05, U1 ProMicro

Commit message: add name and icon, add mounting holes, add trrs support back
Parts:
- added U2: trrs, footprintsGlobal:trrs, symbol keyboard-kicad-lib:trrs
Connections:
- net VCC: now reaches U1.21 (VCC)
- net VCC: now also U2.2 (TIP)
- net GND: now reaches U1.23 (GND)
- net GND: now also U2.3 (RING1)
- net SDA: now reaches U1.5 (SDA)
- net SDA: now also U2.1 (SLEEVE)
Changed lines of the file:
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@@
+    (stroke (width 0) (type default) (color 0 0 0 0))
+  )
+  (wire (pts (xy 213.36 31.75) (xy 210.82 31.75))
     (stroke (width 0) (type default) (color 0 0 0 0))
   )
@@
     (stroke (width 0) (type default) (color 0 0 0 0))
   )
+  (wire (pts (xy 172.72 34.29) (xy 175.26 34.29))
+    (stroke (width 0) (type default) (color 0 0 0 0))
+  )
   (wire (pts (xy 91.44 30.48) (xy 111.76 30.48))
     (stroke (width 0) (type default) (color 0 0 0 0))
@@
   )
   (wire (pts (xy 68.58 30.48) (xy 91.44 30.48))
+    (stroke (width 0) (type default) (color 0 0 0 0))
+  )
+  (wire (pts (xy 210.82 26.67) (xy 213.36 26.67))
     (stroke (width 0) (type default) (color 0 0 0 0))
   )
@@
     )
   )
+  (global_label "GND" (shape input) (at 241.3 29.21 0) (fields_autoplaced)
+    (effects (font (size 1.27 1.27)) (justify left))
+    (property "Intersheet References" "${INTERSHEET_REFS}" (id 0) (at 247.4947 29.1306 0)
+      (effects (font (size 1.27 1.27)) (justify left) hide)
+    )
+  )
   (global_label "CL5" (shape input) (at 201.93 66.04 180) (fields_autoplaced)
     (effects (font (size 1.27 1.27)) (justify right))
@@
     )
   )
+  (global_label "VCC" (shape input) (at 241.3 31.75 0) (fields_autoplaced)
+    (effects (font (size 1.27 1.27)) (justify left))
+    (property "Intersheet References" "${INTERSHEET_REFS}" (id 0) (at 247.2528 31.6706 0)
+      (effects (font (size 1.27 1.27)) (justify left) hide)
+    )
+  )
   (global_label "CR1" (shape input) (at 60.96 17.78 180) (fields_autoplaced)
     (effects (font (size 1.27 1.27)) (justify right))
@@
     )
   )
+  (global_label "VCC" (shape input) (at 213.36 31.75 0) (fields_autoplaced)
+    (effects (font (size 1.27 1.27)) (justify left))
+    (property "Intersheet References" "${INTERSHEET_REFS}" (id 0) (at 219.3128 31.6706 0)
+      (effects (font (size 1.27 1.27)) (justify left) hide)
+    )
+  )
   (global_label "CL2" (shape input) (at 201.93 73.66 180) (fields_autoplaced)
     (effects (font (size 1.27 1.27)) (justify right))
@@
     )
   )
+  (global_label "SDA" (shape input) (at 172.72 34.29 180) (fields_autoplaced)
+    (effects (font (size 1.27 1.27)) (justify right))
+    (property "Intersheet References" "${INTERSHEET_REFS}" (id 0) (at 166.8277 34.2106 0)
+      (effects (font (size 1.27 1.27)) (justify right) hide)
+    )
+  )
   (global_label "CL0" (shape input) (at 219.71 76.2 0) (fields_autoplaced)
     (effects (font (size 1.27 1.27)) (justify left))
@@
     )
   )
+  (global_label "SDA" (shape input) (at 241.3 24.13 0) (fields_autoplaced)
+    (effects (font (size 1.27 1.27)) (justify left))
+    (property "Intersheet References" "${INTERSHEET_REFS}" (id 0) (at 247.1923 24.2094 0)
+      (effects (font (size 1.27 1.27)) (justify left) hide)
+    )
+  )
   (global_label "CL1" (shape input) (at 172.72 41.91 180) (fields_autoplaced)
     (effects (font (size 1.27 1.27)) (justify right))
@@
     (property "Intersheet References" "${INTERSHEET_REFS}" (id 0) (at 0 0 0)
       (effects (font (size 1.27 1.27)) hide)
+    )
+  )
+  (global_label "GND" (shape input) (at 213.36 26.67 0) (fields_autoplaced)
+    (effects (font (size 1.27 1.27)) (justify left))
+    (property "Intersheet References" "${INTERSHEET_REFS}" (id 0) (at 219.5547 26.5906 0)
+      (effects (font (size 1.27 1.27)) (justify left) hide)
     )
   )
@@
     (pin "9")
   )
+  (symbol (lib_id "keyboard-kicad-lib:trrs") (at 232.41 21.59 180) (unit 1)
+    (in_bom yes) (on_board yes) (fields_autoplaced)
+    (property "Reference" "U2" (id 0) (at 231.775 16.51 0)
+      (effects (font (size 1.524 1.524)))
+    )
+    (property "Value" "trrs" (id 1) (at 231.775 20.32 0)
+      (effects (font (size 1.524 1.524)))
+    )
+    (property "Footprint" "footprintsGlobal:trrs" (id 2) (at 228.6 21.59 0)
+      (effects (font (size 1.524 1.524)) hide)
+    )
+    (property "Datasheet" "" (id 3) (at 228.6 21.59 0)
+      (effects (font (size 1.524 1.524)) hide)
+    )
+    (pin "1")
+    (pin "2")
+    (pin "3")
+    (pin "4")
+  )
   (sheet_instances
     (path "/" (page "1"))
@@
       (reference "U1") (unit 1) (value "ProMicro") (footprint "footprints:promicro")
     )
-  )
+    (path "/b64b9c63-ae51-42f0-ac58-38094e4e141c"
+      (reference "U2") (unit 1) (value "trrs") (footprint "footprintsGlobal:trrs")
+    )
+  )

Commit message: add support for smd diodes
Parts:
- D-0-0, D-0-1, D-0-2, D-0-3, D-0-4, D-0-5, D-1-0, D-1-1, D-1-2, D-1-3, D-1-4, D-1-5, D-2-0, D-2-1, D-2-2, D-2-3, D-2-4, D-2-5, D-3-3, D-3-4, D-3-5: footprint footprints:diode-vertical -> footprintsGlobal:Diode-dual
